File: hardware/hat-v1/security.kicad_sch (KiCad schematic)
At the start: 16 parts, among them U11 SLB9672XU20FW1541XTMA1, U12 ATECC608C-TFLXTLS, U13 RV-3028-C7

Commit message: HAT v1 schematic: apply adversarial review (power + digital/security/DFM)
AUTO-ON above buck EN window, BENCH no longer blocks power-off, OVP moved
to 19.2 V with input damper, Tier A parts DNP for JLC, debug links
removable for production, antenna short limited, stock footprints where
available, cap ratings/DC-bias fixes, CONSOLE_TX/RX naming.

Co-Authored-By: Claude Opus 5.5 <noreply@anthropic.com>
Claude-Session: https://claude.ai/code/session_01MLRuxTEmuMV82xcNLE62jW
Parts:
- C76: Note RTC backup -> RTC backup; rated 3.3 V vs 3V3_SEC up to 3.4 V: confirm wit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
- JP5: Note cut to isolate TPM / ATECC / RTC supply -> cut to isolate TPM / ATECC / RTC supply; I2C/SPI1 still bac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; now left out of the parts list
- U11: value SLB9672XU20FW1541XTMA1 -> SLB9672XU2.0; footprint batman:Infineon_PG-UQFN-32-1_5x5mm -> Package_DFN_QFN:QFN-32-1EP_5x5mm_P0.5mm_EP3.6x3.6mm; MPN SLB9672XU2.0 (-40..85C) -> SLB9672XU2.0 (orderable code: verify at M3); now not fitted
- U12: MPN ATECC608C-TFLXTLS-S -> ATECC608C-TFLXTLS (SOIC-8 suffix: verify at M3); now not fitted
- U13: now not fitted
Other:
- note added: "NOTES JP5: cut to isolate TPM / ATECC / RTC supply; I2C/SPI1 still back-power them through ESD diodes U11: NC 6/29/30 must float; GPIO 3/4/7 have internal pull-ups; NO test points on TPM nets C70: pin 1 C71: pin 14 C72: pin 22 R60: pin 10 pull-up (TCG compatibility) R61: datasheet Fig 7: GPIO18 boots pulled down R63: hold TPM in reset until the gpio-hog releases it U12: I2C 0x36 (TrustFLEX) U13: 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"
- note removed: "NOTES JP5: cut to isolate TPM / ATECC / RTC supply U11: NC 6/29/30 must float; GPIO 3/4/7 have internal pull-ups; NO test points on TPM nets C70: pin 1 C71: pin 14 C72: pin 22 R60: pin 10 pull-up (TCG compatibility) R61: datasheet Fig 7: GPIO18 boots pulled down R63: hold TPM in reset until the gpio-hog releases it U12: I2C 0x36 (TrustFLEX) U13: I2C 0x52; trickle charge enabled by the overlay (tr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"
Changed lines of the file:
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@@
   (paper "A4")
   (title_block (title "Batman HAT v1 (Pi 4) - replaces Seeed WM1302 HAT") (date "2026-09-27") (rev "0.1-draft") (company "Batman project - generated by hardware/hat-v1/gen/gen_sch.py, do not edit by hand") (comment 1 "7 TPM 2.0 SLB9672, ATECC608C, RTC RV-3028") (comment 2 "Label-based schematic: same net name = connected"))
-  (symbol (lib_id "batman:SJ") (at 31.75 26.67 0) (unit 1) (in_bom yes) (on_board yes) (dnp no)
+  (symbol (lib_id "batman:SJ") (at 31.75 26.67 0) (unit 1) (in_bom no) (on_board yes) (dnp no)
     (property "Reference" "JP5" (at 31.75 24.13 0) (effects (font (size 1.27 1.27)) (justify bottom)))
     (property "Value" "SEC (closed)" (at 31.75 29.21 0) (effects (font (size 1.27 1.27)) (justify top)))
@@
     (property "Tier" "C" (at 31.75 26.67 0) (effects (font (size 1.27 1.27)) hide))
     (property "LCSC" "" (at 31.75 26.67 0) (effects (font (size 1.27 1.27)) hide))
-    (property "Note" "cut to isolate TPM / ATECC / RTC supply" (at 31.75 26.67 0) (effects (font (size 1.27 1.27)) hide))
+    (property "Note" "cut to isolate TPM / ATECC / RTC supply; I2C/SPI1 still back-power them through ESD diodes" (at 31.75 26.67 0) (effects (font (size 1.27 1.27)) hide))
     (pin "1")
     (pin "2")
@@
   (global_label "3V3_SEC" (shape passive) (at 38.1 26.67 0) (fields_autoplaced) (effects (font (size 1.27 1.27)) (justify left))
     (property "Intersheetrefs" "${INTERSHEET_REFS}" (at 38.1 26.67 0) (effects (font (size 1.27 1.27)) hide)))
-  (symbol (lib_id "batman:SLB9672") (at 88.9 34.29 0) (unit 1) (in_bom yes) (on_board yes) (dnp no)
+  (symbol (lib_id "batman:SLB9672") (at 88.9 34.29 0) (unit 1) (in_bom yes) (on_board yes) (dnp yes)
     (property "Reference" "U11" (at 72.39 24.13 0) (effects (font (size 1.27 1.27)) (justify left bottom)))
-    (property "Value" "SLB9672XU20FW1541XTMA1" (at 72.39 45.72 0) (effects (font (size 1.27 1.27)) (justify left top)))
-    (property "Footprint" "batman:Infineon_PG-UQFN-32-1_5x5mm" (at 88.9 34.29 0) (effects (font (size 1.27 1.27)) hide))
+    (property "Value" "SLB9672XU2.0" (at 72.39 45.72 0) (effects (font (size 1.27 1.27)) (justify left top)))
+    (property "Footprint" "Package_DFN_QFN:QFN-32-1EP_5x5mm_P0.5mm_EP3.6x3.6mm" (at 88.9 34.29 0) (effects (font (size 1.27 1.27)) hide))
     (property "Datasheet" "" (at 88.9 34.29 0) (effects (font (size 1.27 1.27)) hide))
-    (property "MPN" "SLB9672XU2.0 (-40..85C)" (at 88.9 34.29 0) (effects (font (size 1.27 1.27)) hide))
+    (property "MPN" "SLB9672XU2.0 (orderable code: verify at M3)" (at 88.9 34.29 0) (effects (font (size 1.27 1.27)) hide))
     (property "Manufacturer" "Infineon" (at 88.9 34.29 0) (effects (font (size 1.27 1.27)) hide))
     (property "Tier" "A" (at 88.9 34.29 0) (effects (font (size 1.27 1.27)) hide))
@@
   (global_label "GND" (shape passive) (at 160.02 54.61 0) (fields_autoplaced) (effects (font (size 1.27 1.27)) (justify left))
     (property "Intersheetrefs" "${INTERSHEET_REFS}" (at 160.02 54.61 0) (effects (font (size 1.27 1.27)) hide)))
-  (symbol (lib_id "batman:ATECC608") (at 194.31 57.15 0) (unit 1) (in_bom yes) (on_board yes) (dnp no)
+  (symbol (lib_id "batman:ATECC608") (at 194.31 57.15 0) (unit 1) (in_bom yes) (on_board yes) (dnp yes)
     (property "Reference" "U12" (at 187.96 52.07 0) (effects (font (size 1.27 1.27)) (justify left bottom)))
     (property "Value" "ATECC608C-TFLXTLS" (at 187.96 63.5 0) (effects (font (size 1.27 1.27)) (justify left top)))
     (property "Footprint" "Package_SO:SOIC-8_3.9x4.9mm_P1.27mm" (at 194.31 57.15 0) (effects (font (size 1.27 1.27)) hide))
     (property "Datasheet" "" (at 194.31 57.15 0) (effects (font (size 1.27 1.27)) hide))
-    (property "MPN" "ATECC608C-TFLXTLS-S" (at 194.31 57.15 0) (effects (font (size 1.27 1.27)) hide))
+    (property "MPN" "ATECC608C-TFLXTLS (SOIC-8 suffix: verify at M3)" (at 194.31 57.15 0) (effects (font (size 1.27 1.27)) hide))
     (property "Manufacturer" "Microchip" (at 194.31 57.15 0) (effects (font (size 1.27 1.27)) hide))
     (property "Tier" "A" (at 194.31 57.15 0) (effects (font (size 1.27 1.27)) hide))
@@
   (global_label "GND" (shape passive) (at 246.38 54.61 0) (fields_autoplaced) (effects (font (size 1.27 1.27)) (justify left))
     (property "Intersheetrefs" "${INTERSHEET_REFS}" (at 246.38 54.61 0) (effects (font (size 1.27 1.27)) hide)))
-  (symbol (lib_id "batman:RV3028") (at 43.18 77.47 0) (unit 1) (in_bom yes) (on_board yes) (dnp no)
+  (symbol (lib_id "batman:RV3028") (at 43.18 77.47 0) (unit 1) (in_bom yes) (on_board yes) (dnp yes)
     (property "Reference" "U13" (at 31.75 69.85 0) (effects (font (size 1.27 1.27)) (justify left bottom)))
     (property "Value" "RV-3028-C7" (at 31.75 86.36 0) (effects (font (size 1.27 1.27)) (justify left top)))
@@
     (property "Tier" "C" (at 160.02 72.39 0) (effects (font (size 1.27 1.27)) hide))
     (property "LCSC" "" (at 160.02 72.39 0) (effects (font (size 1.27 1.27)) hide))
-    (property "Note" "RTC backup" (at 160.02 72.39 0) (effects (font (size 1.27 1.27)) hide))
+    (property "Note" "RTC backup; rated 3.3 V vs 3V3_SEC up to 3.4 V: confirm with Seiko limit" (at 160.02 72.39 0) (effects (font (size 1.27 1.27)) hide))
     (pin "1")
     (pin "2")
@@
   (global_label "GND" (shape passive) (at 166.37 72.39 0) (fields_autoplaced) (effects (font (size 1.27 1.27)) (justify left))
     (property "Intersheetrefs" "${INTERSHEET_REFS}" (at 166.37 72.39 0) (effects (font (size 1.27 1.27)) hide)))
-  (text "NOTES\nJP5: cut to isolate TPM / ATECC / RTC supply\nU11: NC 6/29/30 must float; GPIO 3/4/7 have internal pull-ups; NO test points on TPM nets\nC70: pin 1\nC71: pin 14\nC72: pin 22\nR60: pin 10 pull-up (TCG compatibility)\nR61: datasheet Fig 7: GPIO18 boots pulled down\nR63: hold TPM in reset until the gpio-hog releases it\nU12: I2C 0x36 (TrustFLEX)\nU13: I2C 0x52; trickle charge enabled by the overlay (trickle-resistor-ohms)\nR64: EVI idle: verify against the RV-3028 Application Manual\nC76: RTC backup" (at 15 93.1 0) (effects (font (size 1.27 1.27)) (justify left top)))
+  (text "NOTES\nJP5: cut to isolate TPM / ATECC / RTC supply; I2C/SPI1 still back-power them through ESD diodes\nU11: NC 6/29/30 must float; GPIO 3/4/7 have internal pull-ups; NO test points on TPM nets\nC70: pin 1\nC71: pin 14\nC72: pin 22\nR60: pin 10 pull-up (TCG compatibility)\nR61: datasheet Fig 7: GPIO18 boots pulled down\nR63: hold TPM in reset until the gpio-hog releases it\nU12: I2C 0x36 (TrustFLEX)\nU13: I2C 0x52; trickle charge enabled by the overlay (trickle-resistor-ohms)\nR64: EVI idle: verify against the RV-3028 Application Manual\nC76: RTC backup; rated 3.3 V vs 3V3_SEC up to 3.4 V: confirm with Seiko limit" (at 15 93.1 0) (effects (font (size 1.27 1.27)) (justify left top)))
 )

Commit message: HAT v1: RV-3028 per Application Manual (land pattern, EVI, VBACKUP 100n, LSM, CLKOUT note)
Co-Authored-By: Claude Opus 5.5 <noreply@anthropic.com>
Claude-Session: https://claude.ai/code/session_01MLRuxTEmuMV82xcNLE62jW
Parts:
- added C77: 100n 16V, Capacitor_SMD:C_0402_1005Metric, symbol batman:C
- C76: Note RTC backup; rated 3.3 V vs 3V3_SEC up to 3.4 V: confirm wit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 -> RTC backup: internal trickle path has a Schottky (0.25 V) -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
- R64: Note EVI idle: verify against the RV-3028 Application Manual -> EVI must not float: tie to VSS through a resistor (App Manu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
- U13: Note I2C 0x52; trickle charge enabled by the overlay (trickle-re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 -> I2C 0x52. App Manual: CLKOUT 32.768 kHz ON by default -> di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
Connections:
- net GND: now also C77.2
- net VRTC: now also C77.1
Changed lines of the file:
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@@
     (property "Tier" "A" (at 43.18 77.47 0) (effects (font (size 1.27 1.27)) hide))
     (property "LCSC" "" (at 43.18 77.47 0) (effects (font (size 1.27 1.27)) hide))
-    (property "Note" "I2C 0x52; trickle charge enabled by the overlay (trickle-resistor-ohms)" (at 43.18 77.47 0) (effects (font (size 1.27 1.27)) hide))
+    (property "Note" "I2C 0x52. App Manual: CLKOUT 32.768 kHz ON by default -> disable in EEPROM (FD=111); backup mode LSM (BSM=11) because VBACKUP ~3.05 V is close to VDD (DSM not recommended, sec 4.2.2)" (at 43.18 77.47 0) (effects (font (size 1.27 1.27)) hide))
     (pin "7")
     (pin "6")
@@
     (property "Tier" "C" (at 128.27 72.39 0) (effects (font (size 1.27 1.27)) hide))
     (property "LCSC" "" (at 128.27 72.39 0) (effects (font (size 1.27 1.27)) hide))
-    (property "Note" "EVI idle: verify against the RV-3028 Application Manual" (at 128.27 72.39 0) (effects (font (size 1.27 1.27)) hide))
+    (property "Note" "EVI must not float: tie to VSS through a resistor (App Manual sec 7.1)" (at 128.27 72.39 0) (effects (font (size 1.27 1.27)) hide))
     (pin "1")
     (pin "2")
@@
     (property "Tier" "C" (at 160.02 72.39 0) (effects (font (size 1.27 1.27)) hide))
     (property "LCSC" "" (at 160.02 72.39 0) (effects (font (size 1.27 1.27)) hide))
-    (property "Note" "RTC backup; rated 3.3 V vs 3V3_SEC up to 3.4 V: confirm with Seiko limit" (at 160.02 72.39 0) (effects (font (size 1.27 1.27)) hide))
+    (property "Note" "RTC backup: internal trickle path has a Schottky (0.25 V) -> charges to ~3.05 V, below the 3.3 V rating. ~2 days backup 3.05->2.0 V at ~60 nA (estimate)" (at 160.02 72.39 0) (effects (font (size 1.27 1.27)) hide))
     (pin "1")
     (pin "2")
@@
   (global_label "GND" (shape passive) (at 166.37 72.39 0) (fields_autoplaced) (effects (font (size 1.27 1.27)) (justify left))
     (property "Intersheetrefs" "${INTERSHEET_REFS}" (at 166.37 72.39 0) (effects (font (size 1.27 1.27)) hide)))
-  (text "NOTES\nJP5: cut to isolate TPM / ATECC / RTC supply; I2C/SPI1 still back-power them through ESD diodes\nU11: NC 6/29/30 must float; GPIO 3/4/7 have internal pull-ups; NO test points on TPM nets\nC70: pin 1\nC71: pin 14\nC72: pin 22\nR60: pin 10 pull-up (TCG compatibility)\nR61: datasheet Fig 7: GPIO18 boots pulled down\nR63: hold TPM in reset until the gpio-hog releases it\nU12: I2C 0x36 (TrustFLEX)\nU13: I2C 0x52; trickle charge enabled by the overlay (trickle-resistor-ohms)\nR64: EVI idle: verify against the RV-3028 Application Manual\nC76: RTC backup; rated 3.3 V vs 3V3_SEC up to 3.4 V: confirm with Seiko limit" (at 15 93.1 0) (effects (font (size 1.27 1.27)) (justify left top)))
+  (symbol (lib_id "batman:C") (at 191.77 72.39 0) (unit 1) (in_bom yes) (on_board yes) (dnp no)
+    (property "Reference" "C77" (at 191.77 69.85 0) (effects (font (size 1.27 1.27)) (justify bottom)))
+    (property "Value" "100n 16V" (at 191.77 74.93 0) (effects (font (size 1.27 1.27)) (justify top)))
+    (property "Footprint" "Capacitor_SMD:C_0402_1005Metric" (at 191.77 72.39 0) (effects (font (size 1.27 1.27)) hide))
+    (property "Datasheet" "" (at 191.77 72.39 0) (effects (font (size 1.27 1.27)) hide))
+    (property "MPN" "" (at 191.77 72.39 0) (effects (font (size 1.27 1.27)) hide))
+    (property "Manufacturer" "" (at 191.77 72.39 0) (effects (font (size 1.27 1.27)) hide))
+    (property "Tier" "C" (at 191.77 72.39 0) (effects (font (size 1.27 1.27)) hide))
+    (property "LCSC" "" (at 191.77 72.39 0) (effects (font (size 1.27 1.27)) hide))
+    (property "Note" "VBACKUP decoupling close to the RTC (App Manual sec 7.3)" (at 191.77 72.39 0) (effects (font (size 1.27 1.27)) hide))
+    (pin "1")
+    (pin "2")
+    (instances (project "batman-hat" (path "/bad0bf22-4662-5834-886f-55d01014b15a/b0ebbc6d-2e97-5070-8b63-d543eba25b44" (reference "C77") (unit 1))))
+  )
+  (wire (pts (xy 187.96 72.39) (xy 185.42 72.39)) (stroke (width 0) (type default)))
+  (global_label "VRTC" (shape passive) (at 185.42 72.39 180) (fields_autoplaced) (effects (font (size 1.27 1.27)) (justify right))
+    (property "Intersheetrefs" "${INTERSHEET_REFS}" (at 185.42 72.39 0) (effects (font (size 1.27 1.27)) hide)))
+  (wire (pts (xy 195.58 72.39) (xy 198.12 72.39)) (stroke (width 0) (type default)))
+  (global_label "GND" (shape passive) (at 198.12 72.39 0) (fields_autoplaced) (effects (font (size 1.27 1.27)) (justify left))
+    (property "Intersheetrefs" "${INTERSHEET_REFS}" (at 198.12 72.39 0) (effects (font (size 1.27 1.27)) hide)))
+  (text "NOTES\nJP5: cut to isolate TPM / ATECC / RTC supply; I2C/SPI1 still back-power them through ESD diodes\nU11: NC 6/29/30 must float; GPIO 3/4/7 have internal pull-ups; NO test points on TPM nets\nC70: pin 1\nC71: pin 14\nC72: pin 22\nR60: pin 10 pull-up (TCG compatibility)\nR61: datasheet Fig 7: GPIO18 boots pulled down\nR63: hold TPM in reset until the gpio-hog releases it\nU12: I2C 0x36 (TrustFLEX)\nU13: I2C 0x52. App Manual: CLKOUT 32.768 kHz ON by default -> disable in EEPROM (FD=111); backup mode LSM (BSM=11) because VBACKUP ~3.05 V is close to VDD (DSM not recommended, sec 4.2.2)\nR64: EVI must not float: tie to VSS through a resistor (App Manual sec 7.1)\nC76: RTC backup: internal trickle path has a Schottky (0.25 V) -> charges to ~3.05 V, below the 3.3 V rating. ~2 days backup 3.05->2.0 V at ~60 nA (estimate)\nC77: VBACKUP decoupling close to the RTC (App Manual sec 7.3)" (at 15 93.1 0) (effects (font (size 1.27 1.27)) (justify left top)))
 )

Commit message: HAT v1: GNSS 3-pin antenna supervisor (UBX-20053088 Fig 38) + RTC coin-cell backup
Antenna supply switched by LNA_EN, 10R sense, OPA333 comparator for open
detection, SCL/SDA reused for ANT_SHORT_N/ANT_DETECT. RTC backup moves to
a Seiko MS rechargeable cell with 1k series resistor (App Manual 7.3);
overlay trickle 15k. Cell footprint does not fit yet (floorplan).

Co-Authored-By: Claude Opus 5.5 <noreply@anthropic.com>
Claude-Session: https://claude.ai/code/session_01MLRuxTEmuMV82xcNLE62jW
Parts:
- removed C76: CPH3225A 11mF, batman:Seiko_CPH3225A, symbol batman:CP
- added BT1: MS621FE 3V 5.5mAh, Battery:BatteryHolder_Seiko_MS621F, symbol batman:BATT
- added R65: 1k, Resistor_SMD:R_0402_1005Metric, symbol batman:R
Connections:
- net GND: now also BT1.2
- net VRTC: now also R65.1
- new net VBAT_RTC: BT1.1, R65.2
Other:
- moved on the sheet: C77

Commit message: HAT v1: keep the CPH3225A supercap for RTC backup (user decision)
Co-Authored-By: Claude Opus 5.5 <noreply@anthropic.com>
Claude-Session: https://claude.ai/code/session_01MLRuxTEmuMV82xcNLE62jW
Parts:
- removed BT1: MS621FE 3V 5.5mAh, Battery:BatteryHolder_Seiko_MS621F, symbol batman:BATT
- removed R65: 1k, Resistor_SMD:R_0402_1005Metric, symbol batman:R
- added C76: CPH3225A 11mF, batman:Seiko_CPH3225A, symbol batman:CP
Connections:
- net GND: now also C76.2
- net VRTC: now also C76.1
Other:
- moved on the sheet: C77
