File: hardware/hat-v1/batman-hat.kicad_pcb (KiCad board)
At the start: 4 copper layers, 65 x 56.5 mm, 174 parts, among them J1 BATT pads, J2 Pi 40-pin (female, 11 mm stac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, J3 mPCIe 5.2H, J4 U.FL, J5 Tag-Connect TC2050, J6 PANEL BTN, Q1 CSD19537Q3, Q10 BSS138, Q11 Si2301CDS, Q12 BSS138, Q2 BSS138, Q3 CSD17578Q3A, Q6 BSS138, Q7 BSS138, U1 TPS26631RGER, U11 SLB9672XU2.0, U12 ATECC608C-TFLXTLS, U13 RV-3028-C7, U14 MAX-M10S-00B, U15 OPA333AIDBVR, U2 INA226AIDGSR, U3 LMR33640DDDAR, U4 LM74700QDBVRQ1, U7 TPS62933FDRLR, U8 INA226AIDGSR, U9 LTC2955ITS8-2#TRPBF

Commit message: HAT v1: nudged GND pads rerouted - 10 unconnected, every GND pad tied to the plane
Co-Authored-By: Claude Opus 5.5 <noreply@anthropic.com>
Claude-Session: https://claude.ai/code/session_01MLRuxTEmuMV82xcNLE62jW
Parts:
- moved C73 0.71 mm to (149.9, 131.0)
- moved Q12 0.25 mm to (142.7, 130.7)
- moved U13 0.25 mm to (127.8, 123.5)
Routing:
- net GND: track 299.5 -> 332.3 mm, vias 148 -> 169
- net VRTC: track 46.1 -> 57.5 mm, vias 4 -> 6
- net PG_5V: track 41.3 -> 31.9 mm
- net HALOW_RESET_N: track 68.2 -> 59.4 mm
- net BAT_PRESENT_N: track 33.6 -> 42.2 mm, vias 1 -> 3
- net GNSS_ANT_DET: track 33.7 -> 28.5 mm
- net 3V3_SEC: track 135.7 -> 140.5 mm
- net VSYS: track 150.3 -> 154.9 mm
- net EF_OUT: track 32.7 -> 37.2 mm, vias 2 -> 3
- net TPM_PIRQ_N: track 44.9 -> 48.2 mm
- net 5V_BUCK: track 103.3 -> 100.7 mm
- net FB_5V: track 16.0 -> 17.8 mm
- net GNSS_ANT_VREF: track 5.49 -> 6.77 mm
- net VCC_5V: track 10.8 -> 9.52 mm
- net KILL_REQ: track 29.1 -> 30.2 mm, vias 1 -> 2
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